File: Phil's_Lab#11.kicad_pcb (KiCad board)
At the start: 4 copper layers, 2 x 7.5 mm, 50 parts, among them J1 Screw_Terminal_01x02, J2 SWD, J3 Conn_01x04, J4 Conn_01x04, J5 USB_B_Micro, Q1 AO3401A, SW1 SW_SPDT, U1 STM32F405RGT6, U3 USBLC6-2SC6, Y1 16MHz

Commit message: .
Parts:
- moved C4 90.2 mm to (118.5, 99.5), turned to -90 degrees
- moved C5 88.0 mm to (126.5, 97.5)
- moved C7 87.0 mm to (127.5, 85.5), turned to 90 degrees
- moved C8 74.8 mm to (113.0, 87.5)
- moved C6 68.7 mm to (117.5, 83.0), turned to 90 degrees
- moved C12 41.9 mm to (66.9, 92.3)
- moved Y1 41.6 mm to (65.5, 89.0)
- moved C11 41.3 mm to (63.9, 92.3)
- moved R2 41.2 mm to (69.9, 88.8)
- moved D4 39.5 mm to (67.4, 101.8)
- moved R11 38.4 mm to (63.4, 101.8), turned to 180 degrees
- moved R1 31.4 mm to (71.0, 73.0)
- moved SW1 31.4 mm to (65.5, 76.0)
- moved J2 29.6 mm to (151.8, 59.5)
- moved U3 28.5 mm to (164.9, 90.0), turned to 180 degrees
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
Commit message: .
Parts:
- moved R8 97.3 mm to (153.3, 100.1), turned to 90 degrees
- moved R6 90.6 mm to (155.2, 100.1), turned to -90 degrees
- moved R7 90.0 mm to (157.2, 100.1), turned to 90 degrees
- moved R5 86.5 mm to (153.3, 96.7), turned to -90 degrees
- moved C15 85.3 mm to (139.4, 107.0)
- moved C14 83.2 mm to (146.6, 99.1), turned to 90 degrees
- moved R4 82.9 mm to (155.3, 96.7), turned to 90 degrees
- moved C16 76.0 mm to (139.4, 109.7)
- moved D2 70.5 mm to (136.3, 88.0), turned to 180 degrees
- moved R12 70.2 mm to (145.2, 83.8)
- moved D5 70.1 mm to (145.7, 82.2)
- moved C13 70.0 mm to (148.7, 95.2), turned to 180 degrees
- moved C10 60.9 mm to (113.6, 93.2), turned to 90 degrees
- moved C3 60.3 mm to (114.4, 83.7), turned to 180 degrees
- moved C9 57.9 mm to (112.5, 93.2), turned to 90 degrees
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Connections:
- F1 pad 1: +12V -> Net-(D3-K)
- F1 pad 2: Net-(Q1-D) -> Net-(F1-Pad2)
- FB1 pad 1: Net-(D3-K) -> Net-(F1-Pad2)
- Q1 pad 3: Net-(Q1-D) -> +12V
Other:
- outline, holes or cut-outs redrawn

Commit message: .
Parts:
- moved H2 123.7 mm to (161.9, 112.0)
- moved H1 108.9 mm to (161.8, 66.0)
- moved H3 75.2 mm to (107.8, 112.0)
- moved H4 50.7 mm to (107.8, 66.0)
- moved SW1 3.07 mm to (107.0, 80.0), turned to -90 degrees
- moved U3 1.83 mm to (158.0, 79.3)
- moved J5 1.83 mm to (167.4, 79.3)
Changed lines of the file:
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@@
 	(footprint "MountingHole:MountingHole_4.3mm_M4_Pad_Via"
 		(layer "F.Cu")
-		(at 57.069581 56.420419)
+		(at 107.775 112)
 		(descr "Mounting Hole 4.3mm, M4, generated by kicad-footprint-generator mountinghole.py")
 		(tags "mountinghole M4")
 		(property "Reference" "H3"
 			(at 0 -5.25 0)
-			(layer "F.SilkS")
+			(layer "F.Fab")
 			(effects
 				(font
@@
 	(footprint "MountingHole:MountingHole_4.3mm_M4_Pad_Via"
 		(layer "F.Cu")
-		(at 57.069581 66.570419)
+		(at 107.8 66)
 		(descr "Mounting Hole 4.3mm, M4, generated by kicad-footprint-generator mountinghole.py")
 		(tags "mountinghole M4")
 		(property "Reference" "H4"
 			(at 0 -5.25 0)
-			(layer "F.SilkS")
+			(layer "F.Fab")
 			(effects
 				(font
@@
 	(footprint "MountingHole:MountingHole_4.3mm_M4_Pad_Via"
 		(layer "F.Cu")
-		(at 57.069581 46.270419)
+		(at 161.855419 112)
 		(descr "Mounting Hole 4.3mm, M4, generated by kicad-footprint-generator mountinghole.py")
 		(tags "mountinghole M4")
 		(property "Reference" "H2"
 			(at 0 -5.25 0)
-			(layer "F.SilkS")
+			(layer "F.Fab")
 			(effects
 				(font
@@
 	(footprint "MountingHole:MountingHole_4.3mm_M4_Pad_Via"
 		(layer "F.Cu")
-		(at 57.069581 36.120419)
+		(at 161.75 66)
 		(descr "Mounting Hole 4.3mm, M4, generated by kicad-footprint-generator mountinghole.py")
 		(tags "mountinghole M4")
 		(property "Reference" "H1"
 			(at 0 -5.25 0)
-			(layer "F.SilkS")
+			(layer "F.Fab")
 			(effects
 				(font
@@
 	(footprint "Connector_USB:USB_Micro-AB_Molex_47590-0001"
 		(layer "F.Cu")
-		(at 165.5575 79.35 90)
+		(at 167.39 79.35 90)
 		(descr "Micro USB AB receptacle, right-angle inverted (https://www.molex.com/pdm_docs/sd/475900001_sd.pdf)")
 		(tags "Micro AB USB SMD")
@@
 	(footprint "Package_TO_SOT_SMD:SOT-23-6"
 		(layer "F.Cu")
-		(at 156.195 79.3 180)
+		(at 158.0275 79.3 180)
 		(descr "SOT, 6 Pin (JEDEC MO-178 Var AB https://www.jedec.org/document_search?search_api_views_fulltext=MO-178), generated with kicad-footprint-generator ipc_gullwing_generator.py")
 		(tags "SOT TO_SOT_SMD")
@@
 	(footprint "Button_Switch_THT:SW_Slide-03_Wuerth-WS-SLTV_10x2.5x6.4_P2.54mm"
 		(layer "F.Cu")
-		(at 104.96 77.75 180)
+		(at 107 80.04 -90)
 		(descr "Wuerth, WS-SLTV, 450301014042, https://www.we-online.com/components/products/datasheet/450301014042.pdf")
 		(tags "switch single-pole opposite-side-connection double-throw SPDT würth wurth")
 		(property "Reference" "SW1"
-			(at 0 -2.54 0)
+			(at 0 -2.54 90)
 			(layer "F.SilkS")
 			(effects
@@
 		)
 		(property "Value" "SW_SPDT"
-			(at 0 3.81 0)
+			(at 0 3.81 90)
 			(layer "F.Fab")
 			(effects
@@
 		)
 		(property "Datasheet" ""
-			(at 0 0 180)
+			(at 0 0 270)
 			(unlocked yes)
 			(layer "F.Fab")
@@
 		)
 		(property "Description" "Switch, single pole double throw"
-			(at 0 0 180)
+			(at 0 0 270)
 			(unlocked yes)
 			(layer "F.Fab")
@@
 		)
 		(fp_text user "${REFERENCE}"
-			(at 0 2.54 0)
+			(at 0 2.54 90)
 			(layer "F.Fab")
 			(effects
@@
 		)
 		(pad "1" thru_hole rect
-			(at 0 0 180)
+			(at 0 0 270)
 			(size 1.5 1.5)
 			(drill 0.8)
@@
 		)
 		(pad "2" thru_hole circle
-			(at -2.54 0 180)
+			(at -2.54 0 270)
 			(size 1.6 1.6)
 			(drill 0.8)
@@
 		)
 		(pad "3" thru_hole circle
-			(at 2.54 0 180)
+			(at 2.54 0 270)
 			(size 1.6 1.6)
 			(drill 0.8)

Commit message: .
Parts:
- moved R12 18.1 mm to (150.0, 66.3), turned to 90 degrees
- moved D5 17.3 mm to (152.0, 66.0), turned to 90 degrees
- moved J3 9.96 mm to (122.0, 65.5)
- moved J4 8.21 mm to (118.2, 112.5)
- moved H1 2.85 mm to (164.6, 66.0)
- moved H2 2.74 mm to (164.6, 112.0)
- moved SW1 2.52 mm to (104.5, 79.7)
- moved J5 1.71 mm to (169.1, 79.3)
- moved U3 0.30 mm to (158.0, 79.0)
Routing:
- added copper zone on In2.Cu, net +3.3V
- added copper zone on In1.Cu, net GND
Other:
- board size 2 x 7.5 mm -> 68 x 57.2 mm
Changed lines of the file:
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@@
 	(footprint "Resistor_SMD:R_0201_0603Metric"
 		(layer "F.Cu")
-		(at 145.23 83.85)
+		(at 150 66.345 90)
 		(descr "Resistor SMD 0201 (0603 Metric), square (rectangular) end terminal, IPC-7351 nominal, (Body size source: https://www.vishay.com/docs/20052/crcw0201e3.pdf), generated with kicad-footprint-generator")
 		(tags "resistor")
 		(property "Reference" "R12"
-			(at 0 -1.05 0)
+			(at 0 -1.05 90)
 			(layer "F.Fab")
 			(effects
@@
 		)
 		(property "Value" "1k"
-			(at 0 1.05 0)
+			(at 0 1.05 90)
 			(layer "F.Fab")
 			(effects
@@
 		)
 		(property "Datasheet" ""
-			(at 0 0 0)
+			(at 0 0 90)
 			(layer "F.Fab")
 			(hide yes)
@@
 		)
 		(property "Description" "Resistor, small symbol"
-			(at 0 0 0)
+			(at 0 0 90)
 			(layer "F.Fab")
 			(hide yes)
@@
 		)
 		(fp_text user "${REFERENCE}"
-			(at 0 -0.68 0)
+			(at 0 -0.68 90)
 			(layer "F.Fab")
 			(effects
@@
 		)
 		(pad "" smd roundrect
-			(at -0.345 0)
+			(at -0.345 0 90)
 			(size 0.318 0.36)
 			(layers "F.Paste")
@@
 		)
 		(pad "" smd roundrect
-			(at 0.345 0)
+			(at 0.345 0 90)
 			(size 0.318 0.36)
 			(layers "F.Paste")
@@
 		)
 		(pad "1" smd roundrect
-			(at -0.32 0)
+			(at -0.32 0 90)
 			(size 0.46 0.4)
 			(layers "F.Cu" "F.Mask")
@@
 		)
 		(pad "2" smd roundrect
-			(at 0.32 0)
+			(at 0.32 0 90)
 			(size 0.46 0.4)
 			(layers "F.Cu" "F.Mask")
@@
 	(footprint "LED_SMD:LED_0603_1608Metric"
 		(layer "F.Cu")
-		(at 145.6875 82.15)
+		(at 152 66 90)
 		(descr "LED SMD 0603 (1608 Metric), square (rectangular) end terminal, IPC-7351 nominal, (Body size source: http://www.tortai-tech.com/upload/download/2011102023233369053.pdf), generated with kicad-footprint-generator")
 		(tags "LED")
 		(property "Reference" "D5"
-			(at 0 -1.43 0)
+			(at 0 -1.43 90)
 			(layer "F.Fab")
 			(effects
@@
 		)
 		(property "Value" "RED"
-			(at 0 1.43 0)
+			(at 0 1.43 90)
 			(layer "F.Fab")
 			(effects
@@
 		)
 		(property "Datasheet" ""
-			(at 0 0 0)
+			(at 0 0 90)
 			(layer "F.Fab")
 			(hide yes)
@@
 		)
 		(property "Description" "Light emitting diode, small symbol"
-			(at 0 0 0)
+			(at 0 0 90)
 			(layer "F.Fab")
 			(hide yes)
@@
 		)
 		(property "Sim.Pins" "1=K 2=A"
-			(at 0 0 0)
+			(at 0 0 90)
 			(unlocked yes)
 			(layer "F.Fab")
@@
 		(duplicate_pad_numbers_are_jumpers no)
 		(fp_line
-			(start -1.485 -0.735)
-			(end -1.485 0.735)
+			(start 0.8 -0.735)
+			(end -1.485 -0.735)
 			(stroke
 				(width 0.12)
@@
 		)
 		(fp_line
-			(start -1.485 0.735)
-			(end 0.8 0.735)
+			(start -1.485 -0.735)
+			(end -1.485 0.735)
 			(stroke
 				(width 0.12)
@@
 		)
 		(fp_line
-			(start 0.8 -0.735)
-			(end -1.485 -0.735)
+			(start -1.485 0.735)
+			(end 0.8 0.735)
 			(stroke
 				(width 0.12)
@@
 		)
 		(fp_line
-			(start -0.8 -0.1)
-			(end -0.8 0.4)
+			(start 0.8 -0.4)
+			(end -0.5 -0.4)
 			(stroke
 				(width 0.1)
@@
 		)
 		(fp_line
-			(start -0.8 0.4)
-			(end 0.8 0.4)
+			(start -0.5 -0.4)
+			(end -0.8 -0.1)
 			(stroke
 				(width 0.1)
@@
 		)
 		(fp_line
-			(start -0.5 -0.4)
-			(end -0.8 -0.1)
+			(start -0.8 -0.1)
+			(end -0.8 0.4)
 			(stroke
 				(width 0.1)
@@
 		)
 		(fp_line
-			(start 0.8 -0.4)
-			(end -0.5 -0.4)
+			(start 0.8 0.4)
+			(end 0.8 -0.4)
 			(stroke
 				(width 0.1)
@@
 		)
 		(fp_line
-			(start 0.8 0.4)
-			(end 0.8 -0.4)
+			(start -0.8 0.4)
+			(end 0.8 0.4)
 			(stroke
 				(width 0.1)
@@
 		)
 		(fp_text user "${REFERENCE}"
-			(at 0 0 0)
+			(at 0 0 90)
 			(layer "F.Fab")
 			(effects
@@
 		)
 		(pad "1" smd roundrect
-			(at -0.7875 0)
+			(at -0.7875 0 90)
 			(size 0.875 0.95)
 			(layers "F.Cu" "F.Mask" "F.Paste")
@@
 		)
 		(pad "2" smd roundrect
-			(at 0.7875 0)
+			(at 0.7875 0 90)
 			(size 0.875 0.95)
 			(layers "F.Cu" "F.Mask" "F.Paste")
@@
 	(footprint "Connector_Molex:Molex_PicoBlade_53048-0410_1x04_P1.25mm_Horizontal"
 		(layer "F.Cu")
-		(at 121.93 75.51 180)
+		(at 122.025 65.55 180)
 		(descr "Molex PicoBlade Connector System, 53048-0410, 4 Pins per row (http://www.molex.com/pdm_docs/sd/530480210_sd.pdf), generated with kicad-footprint-generator")
 		(tags "connector Molex PicoBlade horizontal")
@@
 	(footprint "Connector_Molex:Molex_PicoBlade_53048-0410_1x04_P1.25mm_Horizontal"
 		(layer "F.Cu")
-		(at 118.55 104.3)
+		(at 118.25 112.5)
 		(descr "Molex PicoBlade Connector System, 53048-0410, 4 Pins per row (http://www.molex.com/pdm_docs/sd/530480210_sd.pdf), generated with kicad-footprint-generator")
 		(tags "connector Molex PicoBlade horizontal")
@@
 	(footprint "MountingHole:MountingHole_4.3mm_M4_Pad_Via"
 		(layer "F.Cu")
-		(at 161.855419 112)
+		(at 164.6 112)
 		(descr "Mounting Hole 4.3mm, M4, generated by kicad-footprint-generator mountinghole.py")
 		(tags "mountinghole M4")
@@
 	(footprint "MountingHole:MountingHole_4.3mm_M4_Pad_Via"
 		(layer "F.Cu")
-		(at 161.75 66)
+		(at 164.6 66)
 		(descr "Mounting Hole 4.3mm, M4, generated by kicad-footprint-generator mountinghole.py")
 		(tags "mountinghole M4")
@@
 	(footprint "Connector_USB:USB_Micro-AB_Molex_47590-0001"
 		(layer "F.Cu")
-		(at 167.39 79.35 90)
+		(at 169.1 79.3 90)
 		(descr "Micro USB AB receptacle, right-angle inverted (https://www.molex.com/pdm_docs/sd/475900001_sd.pdf)")
 		(tags "Micro AB USB SMD")
@@
 		(sheetname "/")
 		(sheetfile "Phil's_Lab#11.kicad_sch")
-		(units
-			(unit
-				(name "A")
-				(pins "6" "5" "1" "3" "2" "4")
-			)
-		)
 		(attr smd)
 		(duplicate_pad_numbers_are_jumpers no)
@@
 			(pintype "power_out")
 		)
-		(pad "6" thru_hole oval
+		(pad "SH" thru_hole oval
 			(at -4.175 -0.35 90)
 			(size 1 1.9)
 			(drill oval 0.6 1.3)
-			(property pad_prop_heatsink)
+			(property pad_prop_mechanical)
 			(layers "*.Cu" "*.Mask")
 			(remove_unused_layers no)
@@
 			(pintype "passive+no_connect")
 		)
-		(pad "6" smd rect
+		(pad "SH" smd rect
 			(at -3.7375 -0.35 90)
 			(size 0.875 1.9)
@@
 			(pintype "passive+no_connect")
 		)
-		(pad "6" thru_hole oval
+		(pad "SH" thru_hole oval
 			(at -2.225 -3.35 90)
 			(size 1.05 1.25)
 			(drill oval 0.65 0.85)
-			(property pad_prop_heatsink)
+			(property pad_prop_mechanical)
 			(layers "*.Cu" "*.Mask")
 			(remove_unused_layers no)
@@
 			(pintype "passive+no_connect")
 		)
-		(pad "6" smd roundrect
+		(pad "SH" smd roundrect
 			(at 0 -0.35 90)
 			(size 2.9 1.9)
@@
 			(pintype "passive+no_connect")
 		)
-		(pad "6" thru_hole oval
+		(pad "SH" thru_hole oval
 			(at 2.225 -3.35 90)
 			(size 1.05 1.25)
 			(drill oval 0.65 0.85)
-			(property pad_prop_heatsink)
+			(property pad_prop_mechanical)
 			(layers "*.Cu" "*.Mask")
 			(remove_unused_layers no)
@@
 			(pintype "passive+no_connect")
 		)
-		(pad "6" smd rect
+		(pad "SH" smd rect
 			(at 3.7375 -0.35 90)
 			(size 0.875 1.9)
@@
 			(pintype "passive+no_connect")
 		)
-		(pad "6" thru_hole oval
+		(pad "SH" thru_hole oval
 			(at 4.175 -0.35 90)
 			(size 1 1.9)
 			(drill oval 0.6 1.3)
-			(property pad_prop_heatsink)
+			(property pad_prop_mechanical)
 			(layers "*.Cu" "*.Mask")
 			(remove_unused_layers no)
@@
 		)
 		(embedded_fonts no)
-		(model "${KICAD9_3DMODEL_DIR}/Connector_USB.3dshapes/USB_Micro-AB_Molex_47590-0001.step"
+		(model "${KICAD10_3DMODEL_DIR}/Connector_USB.3dshapes/USB_Micro-AB_Molex_47590-0001.step"
 			(offset
 				(xyz 0 0 0)
@@
 	(footprint "Package_TO_SOT_SMD:SOT-23-6"
 		(layer "F.Cu")
-		(at 158.0275 79.3 180)
+		(at 158.025 79 180)
 		(descr "SOT, 6 Pin (JEDEC MO-178 Var AB https://www.jedec.org/document_search?search_api_views_fulltext=MO-178), generated with kicad-footprint-generator ipc_gullwing_generator.py")
 		(tags "SOT TO_SOT_SMD")
@@
 	(footprint "Button_Switch_THT:SW_Slide-03_Wuerth-WS-SLTV_10x2.5x6.4_P2.54mm"
 		(layer "F.Cu")
-		(at 107 80.04 -90)
+		(at 104.5 79.71 -90)
 		(descr "Wuerth, WS-SLTV, 450301014042, https://www.we-online.com/components/products/datasheet/450301014042.pdf")
 		(tags "switch single-pole opposite-side-connection double-throw SPDT würth wurth")
 		(property "Reference" "SW1"
 			(at 0 -2.54 90)
-			(layer "F.SilkS")
+			(layer "F.Fab")
 			(effects
 				(font
@@
 			)
 		)
+	)
+	(gr_arc
+		(start 102.2 66)
+		(mid 103.840202 62.040202)
+		(end 107.8 60.4)
+		(stroke
+			(width 0.1)
+			(type solid)
+		)
+		(layer "Edge.Cuts")
+	)
+	(gr_line
+		(start 102.2 112)
+		(end 102.2 66)
+		(stroke
+			(width 0.1)
+			(type solid)
+		)
+		(layer "Edge.Cuts")
+	)
+	(gr_line
+		(start 107.8 60.4)
+		(end 164.6 60.4)
+		(stroke
+			(width 0.1)
+			(type solid)
+		)
+		(layer "Edge.Cuts")
+	)
+	(gr_arc
+		(start 107.8 117.6)
+		(mid 103.840202 115.959798)
+		(end 102.2 112)
+		(stroke
+			(width 0.1)
+			(type solid)
+		)
+		(layer "Edge.Cuts")
+	)
+	(gr_arc
+		(start 164.6 60.4)
+		(mid 168.559798 62.040202)
+		(end 170.2 66)
+		(stroke
+			(width 0.1)
+			(type solid)
+		)
+		(layer "Edge.Cuts")
+	)
+	(gr_line
+		(start 164.6 117.6)
+		(end 107.8 117.6)
+		(stroke
+			(width 0.1)
+			(type solid)
+		)
+		(layer "Edge.Cuts")
+	)
+	(gr_line
+		(start 170.2 66)
+		(end 170.2 75.55)
+		(stroke
+			(width 0.05)
+			(type default)
+		)
+		(layer "Edge.Cuts")
+	)
+	(gr_line
+		(start 170.2 83.05)
+		(end 170.2 112)
+		(stroke
+			(width 0.05)
+			(type solid)
+		)
+		(layer "Edge.Cuts")
+	)
+	(gr_arc
+		(start 170.2 112)
+		(mid 168.559798 115.959798)
+		(end 164.6 117.6)
+		(stroke
+			(width 0.1)
+			(type solid)
+		)
+		(layer "Edge.Cuts")
+	)
+	(zone
+		(net "GND")
+		(layer "In1.Cu")
+		(hatch edge 0.5)
+		(connect_pads
+			(clearance 0.5)
+		)
+		(min_thickness 0.25)
+		(fill
+			(thermal_gap 0.5)
+			(thermal_bridge_width 0.5)
+			(island_removal_mode 0)
+		)
+		(polygon
+			(pts
+				(xy 101.5 60) (xy 170.5 60) (xy 170.5 118) (xy 101.5 118)
+			)
+		)
+	)
+	(zone
+		(net "+3.3V")
+		(layer "In2.Cu")
+		(hatch edge 0.5)
+		(connect_pads
+			(clearance 0.5)
+		)
+		(min_thickness 0.25)
+		(fill
+			(thermal_gap 0.5)
+			(thermal_bridge_width 0.5)
+			(island_removal_mode 0)
+		)
+		(polygon
+			(pts
+				(xy 101.5 60) (xy 170.5 60) (xy 170.5 118) (xy 101.5 118)
+			)
+		)

Commit message: .
Parts:
- J5: footprint Connector_USB:USB_Micro-AB_Molex_47590-0001 -> Connector_USB:USB_Micro-B_Amphenol_10118193-0001LF_Horizontal
- moved R1 10.3 mm to (108.4, 77.2)
- moved R12 8.00 mm to (147.5, 73.9)
- moved D5 7.91 mm to (149.5, 73.5)
- moved L2 5.60 mm to (138.0, 103.2)
- moved C15 5.60 mm to (139.5, 112.6)
- moved C16 5.60 mm to (139.5, 115.3)
- moved D2 5.60 mm to (136.4, 93.5)
- moved U3 2.96 mm to (160.6, 80.4)
- moved C11 1.54 mm to (107.9, 86.6)
- moved C12 1.54 mm to (107.9, 92.4)
- moved R2 1.54 mm to (111.5, 90.6)
- moved Y1 1.54 mm to (108.3, 89.5)
- moved C1 1.47 mm to (128.8, 86.7), turned to 90 degrees
- moved J5 0.89 mm to (168.7, 80.1)
- moved R6 0.85 mm to (155.2, 101.0)
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Connections:
- J5 pad SH: unconnected-(J5-Shield-Pad6)_2 -> (no net)
Routing:
- net USB_D-: track 0.00 -> 36.7 mm
- net USB_D+: track 0.00 -> 36.7 mm
- net NRST: track 0.00 -> 32.8 mm, vias 0 -> 2
- net SWO: track 0.00 -> 20.3 mm
- net I2C1_SDA: track 0.00 -> 20.2 mm
- net I2C1_SCL: track 0.00 -> 20.2 mm
- net BOOT0: track 0.00 -> 19.2 mm
- net USART3_TX: track 0.00 -> 17.2 mm
- net USART3_RX: track 0.00 -> 16.9 mm
- net +3.3V: track 0.00 -> 16.7 mm
- net SWDIO: track 0.00 -> 15.9 mm, vias 0 -> 2
- net BUCK_SW: track 0.00 -> 15.4 mm
- net SWCLK: track 0.00 -> 12.9 mm
- net HSE_IN: track 0.00 -> 10.8 mm
- net +5V: track 0.00 -> 9.46 mm
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Other:
- outline, holes or cut-outs redrawn
