File: Phil's_Lab#11.kicad_pcb (KiCad board)
At the start: 4 copper layers, 68 x 57.2 mm, 50 parts, among them J1 Screw_Terminal_01x02, J2 SWD, J3 Conn_01x04, J4 Conn_01x04, J5 USB_B_Micro, Q1 AO3401A, SW1 SW_SPDT, U1 STM32F405RGT6, U3 USBLC6-2SC6, Y1 16MHz

Commit message: .
Routing:
- net GND: track 8.65 -> 47.0 mm, vias 0 -> 36
- net +3.3V: track 16.7 -> 29.4 mm, vias 0 -> 23
- net +5V: track 9.46 -> 18.7 mm
- added copper zone on F.Cu, net +3.3V

Commit message: .
Parts:
- J2: footprint Connector_PinSocket_1.27mm:PinSocket_2x05_P1.27mm_Vertical_SMD -> Connector_PinHeader_1.27mm:PinHeader_2x05_P1.27mm_Vertical_SMD
- moved J2 1.50 mm to (132.3, 73.1), turned to -90 degrees
Routing:
- net NRST: track 32.8 -> 22.4 mm
- net GND: track 47.0 -> 52.1 mm, vias 36 -> 40
- net SWDIO: track 15.9 -> 19.6 mm, vias 2 -> 0
- net SWCLK: track 12.9 -> 14.1 mm
- net SWO: track 20.3 -> 21.1 mm
Other:
- board text added: "+"
- board text added: "3.3V"
- board text added: "BOOT"
- board text added: "DEBUG"
- board text added: "I2C"
- board text added: "JLCJLCJLCJLC"
- board text added: "LED"
- board text added: "POWER"
- board text added: "UART"
- board text added: "USB"
